File: circuito/design/sensor.kicad_pcb (KiCad board)
At the start: 2 copper layers, 50 x 50 mm, 9 parts

Commit message: Implementación con 7805
Parts:
- removed VIN1: CONN_01X02, Connectors_Molex:Molex_KK_6410-02
- added U1: 7805, TO_SOT_Packages_THT:TO-220_Neutral123_Vertical, F.Cu at (108.7, 140.1)
Connections:
- MC1 pad 9: Net-(MC1-Pad9) -> (no net)
- RV1 pad 3: Net-(RV1-Pad3) -> (no net)
- uC1 pad 10: Net-(uC1-Pad10) -> (no net)
- uC1 pad 11: Net-(uC1-Pad11) -> (no net)
- uC1 pad 15: Net-(uC1-Pad15) -> (no net)
- uC1 pad 16: Net-(uC1-Pad16) -> (no net)
- uC1 pad 17: Net-(uC1-Pad17) -> (no net)
- uC1 pad 22: Net-(uC1-Pad22) -> (no net)
- uC1 pad 23: Net-(uC1-Pad23) -> (no net)
- uC1 pad 3: Net-(uC1-Pad3) -> (no net)
- uC1 pad 4: Net-(uC1-Pad4) -> (no net)
- uC1 pad 5: Net-(uC1-Pad5) -> (no net)
- uC1 pad 6: Net-(uC1-Pad6) -> (no net)
- uC1 pad 7: Net-(uC1-Pad7) -> (no net)
- uC1 pad 8: Net-(uC1-Pad8) -> (no net)
- uC1 pad 9: Net-(uC1-Pad9) -> (no net)
Routing:
- net +12V: track 13.5 -> 29.0 mm
- net +5V: track 121.6 -> 126.7 mm
Other:
- outline, holes or cut-outs redrawn
