File: circuito/design/sensor.sch (KiCad schematic (older format))
At the start: 9 parts

Commit message: Implementación con 7805
Parts:
- removed VIN1: CONN_01X02, Connectors_Molex:Molex_KK_6410-02, symbol CONN_01X02
- added U1: 7805, Power_Integrations:TO-220, symbol 7805
Connections:
- wire segments 55 -> 56
Changed lines of the file:
@@
 LIBS:particle-boards
 LIBS:pololu_a4988
+LIBS:sensor-cache
 EELAYER 25 0
 EELAYER END
@@
 	6950 5200 6950 5100
 $Comp
-L CONN_01X02 VIN1
-U 1 1 5752FE54
-P 5350 3450
-F 0 "VIN1" H 5350 3600 50  0000 C CNN
-F 1 "CONN_01X02" V 5450 3450 50  0000 C CNN
-F 2 "Connectors_Molex:Molex_KK_6410-02" H 5350 3450 50  0001 C CNN
-F 3 "" H 5350 3450 50  0000 C CNN
-	1    5350 3450
-	1    0    0    -1
-$EndComp
-$Comp
-L +5V #PWR020
-U 1 1 5752FF99
-P 5050 3200
-F 0 "#PWR020" H 5050 3050 50  0001 C CNN
-F 1 "+5V" H 5050 3340 50  0000 C CNN
-F 2 "" H 5050 3200 50  0000 C CNN
-F 3 "" H 5050 3200 50  0000 C CNN
-	1    5050 3200
-	1    0    0    -1
-$EndComp
-$Comp
-L GND #PWR021
-U 1 1 57530031
-P 5050 3600
-F 0 "#PWR021" H 5050 3350 50  0001 C CNN
-F 1 "GND" H 5050 3450 50  0000 C CNN
-F 2 "" H 5050 3600 50  0000 C CNN
-F 3 "" H 5050 3600 50  0000 C CNN
-	1    5050 3600
-	1    0    0    -1
-$EndComp
-Wire Wire Line
-	5150 3400 5050 3400
-Wire Wire Line
-	5050 3400 5050 3200
-Wire Wire Line
-	5150 3500 5050 3500
-Wire Wire Line
-	5050 3500 5050 3600
+L 7805 U1
+U 1 1 5814FDFB
+P 5400 2650
+F 0 "U1" H 5550 2454 50  0000 C CNN
+F 1 "7805" H 5400 2850 50  0000 C CNN
+F 2 "Power_Integrations:TO-220" H 5400 2650 50  0001 C CNN
+F 3 "" H 5400 2650 50  0000 C CNN
+	1    5400 2650
+	1    0    0    -1
+$EndComp
+$Comp
+L +12V #PWR020
+U 1 1 5814FFDF
+P 4850 2500
+F 0 "#PWR020" H 4850 2350 50  0001 C CNN
+F 1 "+12V" H 4850 2640 50  0000 C CNN
+F 2 "" H 4850 2500 50  0000 C CNN
+F 3 "" H 4850 2500 50  0000 C CNN
+	1    4850 2500
+	1    0    0    -1
+$EndComp
+$Comp
+L +5V #PWR021
+U 1 1 58150134
+P 5850 2450
+F 0 "#PWR021" H 5850 2300 50  0001 C CNN
+F 1 "+5V" H 5850 2590 50  0000 C CNN
+F 2 "" H 5850 2450 50  0000 C CNN
+F 3 "" H 5850 2450 50  0000 C CNN
+	1    5850 2450
+	1    0    0    -1
+$EndComp
+$Comp
+L GND #PWR022
+U 1 1 5815015D
+P 5400 3000
+F 0 "#PWR022" H 5400 2750 50  0001 C CNN
+F 1 "GND" H 5400 2850 50  0000 C CNN
+F 2 "" H 5400 3000 50  0000 C CNN
+F 3 "" H 5400 3000 50  0000 C CNN
+	1    5400 3000
+	1    0    0    -1
+$EndComp
+Wire Wire Line
+	4850 2500 4850 2600
+Wire Wire Line
+	4850 2600 5000 2600
+Wire Wire Line
+	5400 2900 5400 3000
+Wire Wire Line
+	5800 2600 5850 2600
+Wire Wire Line
+	5850 2600 5850 2450
 $EndSCHEMATC
